File: test/fixtures/footprint-enumerator/board-with-footprints.kicad_pcb (KiCad board)
At the start: 2 parts

Commit message: feat: update s-expression tooling and add new footprint to test fixtures
Parts:
- added J1: Conn_01x02, Connector_PinHeader_2.00mm:PinHeader_1x2_P2.00mm_Vertical, F.Cu at (135.0, 90.0)
Changed lines of the file:
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@@
     (property "Value" "1uF")
   )
+  (footprint "Connector_PinHeader_2.00mm:PinHeader_1x2_P2.00mm_Vertical"
+    (at 135 90 0)
+    (property "Reference" "J1")
+    (property "Value" "Conn_01x02")
+  )
 )
