File: test/fixtures/open-key/hardware/open-key.kicad_sch (KiCad schematic)
At the start: 3 parts, among them U1 ESP32-S3-MINI

Commit message: feat(kicad): implement the legibility checker phase (groups 1-4 of deterministic-schematic-drafting)
Read-only geometry accessors in sexp.ts (sheet graphics, labels, wires, paper,
title block, lib body bounds); src/kicad/legibility.ts with the 13 check
families, conservative text extents, per-family caps with stated suppression,
and the optional legibility config block; check_legibility agent tool feeding
a new ledger obligation that finish enforces; drafting-standard block and
reconcile instruction in the stage-4 prompt; legibility joins the schematic
stage completion contract with finding counts in the halt message and counts
recorded in run summaries; check reports findings advisory-only and check
--json gains the legibility object (score reserved as null).

Label text boxes are direction-aware (they extend away from the anchor, as
eeschema renders them) so the checker cannot invent collisions with the
symbol a label serves - the C3 under-estimate rule. The open-key fixture is
upgraded to the drafting standard (captioned group box, dated title block);
new clean/ugly/hierarchical fixtures exercise every family.

AC covered: 16.22, 16.25, 16.27-16.30. 598 tests pass.

Co-Authored-By: Claude Fable 5 <noreply@anthropic.com>
Other:
- note added: "Keyer"
Changed lines of the file:
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@@
   (title_block
     (title "open-key fixture")
+    (date "2026-07-31")
     (rev "A")
     (comment 1 "Minimal copperhead test fixture")
@@
   (no_connect (at 127 104.14))
   (no_connect (at 127 106.68))
+  (rectangle (start 80 84) (end 160 120)
+    (stroke (width 0.152) (type solid))
+    (fill (type none))
+    (uuid "0f0f0f0f-0000-4000-8000-00000000r001")
+  )
+  (text "Keyer" (at 85 87.5 0)
+    (effects (font (size 2 2)))
+    (uuid "0f0f0f0f-0000-4000-8000-00000000t001")
+  )
   (global_label "3V3" (shape input) (at 127 91.44 180) (fields_autoplaced yes)
     (effects (font (size 1.27 1.27)) (justify right))
